File: vfo-do/vfo-do.kicad_pcb (KiCad board)
At the start: 2 copper layers, 19 parts, among them J1 Fréquence, J10 GPS, J2 Bande, J3 Reset, J4 Résolution, J5 Si5351, J6 Contraste, J7 Backlight, J8 LCD, J9 Alim +12V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

Commit message: Nouveau design PCB avec les conseils du discord
Parts:
- removed J6: Contraste, Connector_PinHeader_2.54mm:PinHeader_1x03_P2.54mm_Vertical
- removed J7: Backlight, Connector_PinHeader_2.54mm:PinHeader_1x02_P2.54mm_Vertical
- added RV1: Contraste, Potentiometer_SMD:Potentiometer_Vishay_TS53YL_Vertical, F.Cu at (82.5, 44.5)
- added RV2: Backlight, Potentiometer_SMD:Potentiometer_Vishay_TS53YL_Vertical, F.Cu at (139.7, 44.5)
- C3, C4, C5, C6, D1, U1: moved to F.Cu
- moved J4 47.0 mm to (81.3, 52.1)
- moved J5 24.7 mm to (81.3, 57.1)
- moved J3 23.3 mm to (139.7, 54.6)
- moved J2 21.5 mm to (81.3, 77.5), turned to 90 degrees
- moved C6 21.1 mm to (114.6, 73.9)
- moved C3 20.7 mm to (114.6, 78.5)
- moved U1 20.4 mm to (101.4, 76.2), turned to 180 degrees
- moved A1 18.9 mm to (127.0, 52.1)
- moved D1 18.7 mm to (120.7, 76.2), turned to 90 degrees
- moved C5 17.0 mm to (110.0, 73.9)
- moved C4 16.5 mm to (110.0, 78.5)
- moved J8 16.3 mm to (92.7, 43.2)
- moved J9 13.6 mm to (125.5, 77.2), turned to 180 degrees
- moved J10 11.1 mm to (139.7, 77.5), turned to 180 degrees
- moved C2 9.25 mm to (134.6, 63.5), turned to 90 degrees
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Connections:
- net K renamed GND
Routing:
- net +5V: track 0.00 -> 139.8 mm
- net CLK0: track 0.00 -> 46.0 mm
- net PPS: track 0.00 -> 43.5 mm
- net RotaryA: track 0.00 -> 35.1 mm, vias 0 -> 1
- net D7: track 0.00 -> 35.0 mm
- net D6: track 0.00 -> 35.0 mm
- net D5: track 0.00 -> 35.0 mm
- net D4: track 0.00 -> 35.0 mm
- net RotaryB: track 0.00 -> 34.8 mm
- net GPS_RX: track 0.00 -> 34.6 mm
- net SCL: track 0.00 -> 32.3 mm, vias 0 -> 1
- net SDA: track 0.00 -> 32.3 mm
- net Bande: track 0.00 -> 30.0 mm
- net Résolution: track 0.00 -> 26.5 mm
- net RST: track 0.00 -> 20.8 mm
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- added copper zone on B.Cu, net GND
- added copper zone on F.Cu, net GND
