File: vfo-do/trimmer-boutons-regroupés/vfo-do-with-trimmer_boutons regroupés.kicad_pcb (KiCad board)
At the start: 2 copper layers, 81 x 44 mm, 23 parts, among them J1 Fréquence, J10 GPS, J2 Bande, J3 Reset, J4 Résolution, J5 Si5351, J8 LCD, J9 Alim +12V, U1 L7805

Commit message: plaque standard 10x5
Parts:
- removed REF** (x4): MountingHole_3.2mm_M3_Pad_Via, MountingHole:MountingHole_3.2mm_M3_Pad_Via
- added TP1: TestPoint_Alt, MountingHole:MountingHole_3.2mm_M3_Pad_Via, F.Cu at (74.5, 43.5)
- added TP2: TestPoint_Alt, MountingHole:MountingHole_3.2mm_M3_Pad_Via, F.Cu at (144.3, 76.4)
- added TP3: TestPoint_Alt, MountingHole:MountingHole_3.2mm_M3_Pad_Via, F.Cu at (144.4, 43.5)
- added TP4: TestPoint_Alt, MountingHole:MountingHole_3.2mm_M3_Pad_Via, F.Cu at (74.7, 76.3)
