File: vfo-do/trimmer-boutons-regroupés-10x5/vfo-do-with-trimmer_boutons regroupés-10x5.kicad_pcb (KiCad board)
At the start: 2 copper layers, 100 x 50 mm, 23 parts, among them J1 Fréquence, J10 GPS, J2 Bande, J3 Reset, J4 Résolution, J5 Si5351, J8 LCD, J9 Alim +12V, U1 L7805

Commit message: Ajout des bonnes empreintes pour les trimmers
Parts:
- added REF**: OSHW-Logo2_9.8x8mm_SilkScreen, Symbol:OSHW-Logo2_9.8x8mm_SilkScreen, B.Cu at (185.0, 139.0)
- RV1, RV2: footprint Potentiometer_SMD:Potentiometer_Vishay_TS53YL_Vertical -> rfa_trimmer:trimmer_3x3
- moved RV1 3.34 mm to (130.8, 105.4), turned to 0 degrees
- moved RV2 3.34 mm to (116.8, 105.4), turned to 0 degrees
Routing:
- net SCL: track 0.00 -> 49.3 mm
- net SDA: track 0.00 -> 49.3 mm, vias 0 -> 1
- net +5V: track 153.4 -> 159.6 mm
- net CLK0: track 50.1 -> 48.7 mm
- net D4: track 33.2 -> 34.2 mm
- net D6: track 33.4 -> 34.2 mm
- net D7: track 33.4 -> 34.2 mm
- net D5: track 33.4 -> 34.2 mm
Other:
- board text added: "Backlight"
- board text added: "Bande"
- board text added: "Contraste"
- board text added: "Fréq."
- board text added: "GPS"
- board text added: "LCD"
- board text added: "Oscillateur à fréquence variable (VFO) Richard Fagot, Sept. 2020 Schéma de W3PM"
- board text added: "Oscillateur à fréquence variable (VFO) à signaux carrés, asservi par GPS."
- board text added: "Reset"
- board text added: "Rés."
- board text added: "Si5351"
