File: kicad/vfo-do-W3PM.kicad_pcb (KiCad board)
At the start: 2 copper layers, 100 x 50 mm, 24 parts, among them J1 Fréquence, J10 GPS, J2 Bande, J3 Reset, J4 Résolution, J5 Si5351, J8 LCD, J9 Alim +12V, U1 L7805

Commit message: Réorganisation du projet + début doc
Parts:
- moved REF** 8.50 mm to (177.8, 143.5)
Other:
- board text added: "+5"
- board text added: "Bouton"
- board text added: "CLK0"
- board text added: "Encodeur Rot."
- board text added: "GND"
- board text added: "Oscillateur à fréquence variable (VFO-DO) Richard Fagot, Sept. 2020 Schéma de W3PM https://github.com/richard-fagot/ra-w3pm-vfo-do"
- board text added: "PPS"
- board text added: "RX"
- board text added: "SCL"
- board text added: "SDA"
- board text added: "https://github.com/richard-fagot/ra-w3pm-vfo-do"
- board text removed: "Oscillateur à fréquence variable (VFO) Richard Fagot, Sept. 2020 Schéma de W3PM"

Commit message: Fix sens connecteur LCD
Parts:
- removed REF**: OSHW-Logo2_9.8x8mm_SilkScreen, Symbol:OSHW-Logo2_9.8x8mm_SilkScreen
- TP1, TP2, TP3, TP4: value TestPoint_Alt -> Fixation
- moved J8 35.7 mm to (184.2, 106.0), turned to 90 degrees
- moved J9 1.70 mm to (185.7, 143.5)
- moved U1 0.14 mm to (151.1, 141.2)
Connections:
- A1 pad 12: D7 -> D4
- A1 pad 13: D6 -> D5
- A1 pad 14: D5 -> D6
- A1 pad 15: D4 -> D7
Routing:
- net A: track 71.2 -> 35.3 mm, vias 0 -> 1
- net V0: track 25.8 -> 50.9 mm
- net D7: track 34.2 -> 9.88 mm
- net D4: track 34.2 -> 9.88 mm
- net D6: track 34.2 -> 9.88 mm
- net D5: track 34.2 -> 10.6 mm
- net RS: track 8.86 -> 24.7 mm
- net E: track 8.79 -> 17.1 mm
- net RotaryB: track 32.7 -> 37.2 mm, vias 0 -> 2
- net RotaryA: track 29.2 -> 32.2 mm, vias 0 -> 2
- net +5V: track 159.6 -> 162.2 mm
- net +12V: track 7.58 -> 6.14 mm
- net CLK0: track 48.7 -> 49.8 mm
- net RST: track 20.6 -> 21.5 mm
- net PPS: track 70.5 -> 71.2 mm
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Other:
- board text added: "+5V"
- board text added: "A"
- board text added: "Alim 10-12V"
- board text added: "CLK1"
- board text added: "CLK2"
- board text added: "D0"
- board text added: "D1"
- board text added: "D2"
- board text added: "D3"
- board text added: "D4"
- board text added: "D5"
- board text added: "D6"
- board text added: "D7"
- board text added: "E"
- board text added: "K"
- board text added: "Oscillateur à fréquence variable (VFO) à signaux carrés, asservi par GPS. V1.1"
- board text added: "Oscillateur à fréquence variable (VFO-DO) V1.1 Richard Fagot, Sept. 2020 Schéma de W3PM https://github.com/richard-fagot/ra-w3pm-vfo-do"
- board text added: "RS"
- board text added: "RW"
- board text added: "V0"
- board text added: "VDD"
- board text added: "VSS"
- board text removed: "Oscillateur à fréquence variable (VFO) à signaux carrés, asservi par GPS."
- board text removed: "Oscillateur à fréquence variable (VFO-DO) Richard Fagot, Sept. 2020 Schéma de W3PM https://github.com/richard-fagot/ra-w3pm-vfo-do"
- board text removed: "https://github.com/richard-fagot/ra-w3pm-vfo-do"
